File: EnvOpenSensor/EnvOpenSensor.kicad_pcb (KiCad board)
At the start: 2 copper layers, 89.7 x 67.5 mm, 31 parts, among them J1 USB_C_Receptacle_USB2.0_16P, J2 AVR-ISP-6, SW1 SW_Push, SW2 SW_Push, SW3 SW_Push, SW4 SW_Push, U1 SCD41-D-R2, U2 Si7021-A20, U3 SPX3819M5-L-3-3, U4 ATtiny85-20S

Commit message: commit current version
Parts:
- added C0: 0402 0.1uF, Capacitor_SMD:C_0402_1005Metric, F.Cu at (67.8, 43.2)
- added C10: 0402 0.1uF, Capacitor_SMD:C_0402_1005Metric, F.Cu at (95.3, 43.2)
- added C11: 0402 0.1uF, Capacitor_SMD:C_0402_1005Metric, F.Cu at (77.2, 43.2)
- added C12: 0402 1uF, Capacitor_SMD:C_0402_1005Metric, F.Cu at (95.3, 44.2)
- added C13: 0402 1uF, Capacitor_SMD:C_0402_1005Metric, F.Cu at (77.2, 44.2)
- added C14: 0402 10uF, Capacitor_SMD:C_0402_1005Metric, F.Cu at (95.3, 45.2)
- added C15: 0402 10uF, Capacitor_SMD:C_0402_1005Metric, F.Cu at (77.2, 45.2)
- added C5: 0402 0.1uF, Capacitor_SMD:C_0402_1005Metric, F.Cu at (86.2, 43.2)
- added C6: 0402 1uF, Capacitor_SMD:C_0402_1005Metric, F.Cu at (67.8, 44.2)
- added C7: 0402 1uF, Capacitor_SMD:C_0402_1005Metric, F.Cu at (86.2, 44.2)
- added C8: 0402 10uF, Capacitor_SMD:C_0402_1005Metric, F.Cu at (67.8, 45.2)
- added C9: 0402 10uF, Capacitor_SMD:C_0402_1005Metric, F.Cu at (86.2, 45.2)
- added IC1: IS31FL3730-QFLS2-TR, Package_DFN_QFN:QFN-24-1EP_4x4mm_P0.5mm_EP2.6x2.6mm_ThermalVias, F.Cu at (66.6, 40.0)
- added IC2: IS31FL3730-QFLS2-TR, Package_DFN_QFN:QFN-24-1EP_4x4mm_P0.5mm_EP2.6x2.6mm_ThermalVias, F.Cu at (76.0, 40.0)
- added IC3: IS31FL3730-QFLS2-TR, Package_DFN_QFN:QFN-24-1EP_4x4mm_P0.5mm_EP2.6x2.6mm_ThermalVias, F.Cu at (85.0, 40.0)
- added IC4: IS31FL3730-QFLS2-TR, Package_DFN_QFN:QFN-24-1EP_4x4mm_P0.5mm_EP2.6x2.6mm_ThermalVias, F.Cu at (94.1, 40.0)
- added NT0: NetTie_2, NetTie:NetTie-2_SMD_Pad0.5mm, F.Cu at (59.7, 43.0)
- H1, H2, H3, H4: value MountingHole -> DIY-305-ountingHole
- U3: value SPX3819M5-L-3-3 -> SPX3819DIY-305-5-L-3-3
Connections:
- DIY-305-0 pad 1: unconnected-(DIY-305-0-Col2-Pad1) -> IC2C2
- DIY-305-0 pad 10: unconnected-(DIY-305-0-Row6-Pad10) -> IC2R6
- DIY-305-0 pad 11: unconnected-(DIY-305-0-Row5-Pad11) -> IC2R5
- DIY-305-0 pad 12: unconnected-(DIY-305-0-Row2-Pad12) -> IC2R2
- DIY-305-0 pad 13: unconnected-(DIY-305-0-Col5-Pad13) -> IC2C5
- DIY-305-0 pad 14: unconnected-(DIY-305-0-Col4-Pad14) -> IC2C4
- DIY-305-0 pad 2: unconnected-(DIY-305-0-Row1-Pad2) -> IC2R1
- DIY-305-0 pad 3: unconnected-(DIY-305-0-Row3-Pad3) -> IC2R3
- DIY-305-0 pad 4: unconnected-(DIY-305-0-Row4-Pad4) -> IC2R4
- DIY-305-0 pad 5: unconnected-(DIY-305-0-Col1-Pad5) -> IC2C1
- DIY-305-0 pad 7: unconnected-(DIY-305-0-Dot-Pad7) -> IC2C8
- DIY-305-0 pad 8: unconnected-(DIY-305-0-Col3-Pad8) -> IC2C3
- DIY-305-0 pad 9: unconnected-(DIY-305-0-Row7-Pad9) -> IC2R7
- DIY-305-1 pad 1: unconnected-(DIY-305-1-Col2-Pad1) -> IC2R2
- DIY-305-1 pad 10: unconnected-(DIY-305-1-Row6-Pad10) -> IC2C6
- DIY-305-1 pad 11: unconnected-(DIY-305-1-Row5-Pad11) -> IC2C5
- DIY-305-1 pad 12: unconnected-(DIY-305-1-Row2-Pad12) -> IC2C2
- DIY-305-1 pad 13: unconnected-(DIY-305-1-Col5-Pad13) -> IC2R5
- DIY-305-1 pad 14: unconnected-(DIY-305-1-Col4-Pad14) -> IC2R4
- DIY-305-1 pad 2: unconnected-(DIY-305-1-Row1-Pad2) -> IC2C1
- DIY-305-1 pad 3: unconnected-(DIY-305-1-Row3-Pad3) -> IC2C3
- DIY-305-1 pad 4: unconnected-(DIY-305-1-Row4-Pad4) -> IC2C4
- DIY-305-1 pad 5: unconnected-(DIY-305-1-Col1-Pad5) -> IC2R1
- DIY-305-1 pad 7: unconnected-(DIY-305-1-Dot-Pad7) -> IC2R8
- DIY-305-1 pad 8: unconnected-(DIY-305-1-Col3-Pad8) -> IC2R3
- DIY-305-1 pad 9: unconnected-(DIY-305-1-Row7-Pad9) -> IC2C7
- DIY-305-2 pad 1: unconnected-(DIY-305-2-Col2-Pad1) -> IC1C2
- DIY-305-2 pad 10: unconnected-(DIY-305-2-Row6-Pad10) -> IC1R6
- DIY-305-2 pad 11: unconnected-(DIY-305-2-Row5-Pad11) -> IC1R5
- DIY-305-2 pad 12: unconnected-(DIY-305-2-Row2-Pad12) -> IC1R2
- DIY-305-2 pad 13: unconnected-(DIY-305-2-Col5-Pad13) -> IC1C5
- DIY-305-2 pad 14: unconnected-(DIY-305-2-Col4-Pad14) -> IC1C4
- DIY-305-2 pad 2: unconnected-(DIY-305-2-Row1-Pad2) -> IC1R1
- DIY-305-2 pad 3: unconnected-(DIY-305-2-Row3-Pad3) -> IC1R3
- DIY-305-2 pad 4: unconnected-(DIY-305-2-Row4-Pad4) -> IC1R4
- DIY-305-2 pad 5: unconnected-(DIY-305-2-Col1-Pad5) -> IC1C1
- DIY-305-2 pad 7: unconnected-(DIY-305-2-Dot-Pad7) -> IC1C8
- DIY-305-2 pad 8: unconnected-(DIY-305-2-Col3-Pad8) -> IC1C3
- DIY-305-2 pad 9: unconnected-(DIY-305-2-Row7-Pad9) -> IC1R7
- DIY-305-3 pad 1: unconnected-(DIY-305-3-Col2-Pad1) -> IC1R2
- DIY-305-3 pad 10: unconnected-(DIY-305-3-Row6-Pad10) -> IC1C6
- DIY-305-3 pad 11: unconnected-(DIY-305-3-Row5-Pad11) -> IC1C5
- DIY-305-3 pad 12: unconnected-(DIY-305-3-Row2-Pad12) -> IC1C2
- DIY-305-3 pad 13: unconnected-(DIY-305-3-Col5-Pad13) -> IC1R5
- DIY-305-3 pad 14: unconnected-(DIY-305-3-Col4-Pad14) -> IC1R4
- DIY-305-3 pad 2: unconnected-(DIY-305-3-Row1-Pad2) -> IC1C1
- DIY-305-3 pad 3: unconnected-(DIY-305-3-Row3-Pad3) -> IC1C3
- DIY-305-3 pad 4: unconnected-(DIY-305-3-Row4-Pad4) -> IC1C4
- DIY-305-3 pad 5: unconnected-(DIY-305-3-Col1-Pad5) -> IC1R1
- DIY-305-3 pad 7: unconnected-(DIY-305-3-Dot-Pad7) -> IC1R8
- DIY-305-3 pad 8: unconnected-(DIY-305-3-Col3-Pad8) -> IC1R3
- DIY-305-3 pad 9: unconnected-(DIY-305-3-Row7-Pad9) -> IC1C7
- DIY-305-4 pad 1: unconnected-(DIY-305-4-Col2-Pad1) -> IC3C2
- DIY-305-4 pad 10: unconnected-(DIY-305-4-Row6-Pad10) -> IC3R6
- DIY-305-4 pad 11: unconnected-(DIY-305-4-Row5-Pad11) -> IC3R5
- DIY-305-4 pad 12: unconnected-(DIY-305-4-Row2-Pad12) -> IC3R2
- DIY-305-4 pad 13: unconnected-(DIY-305-4-Col5-Pad13) -> IC3C5
- DIY-305-4 pad 14: unconnected-(DIY-305-4-Col4-Pad14) -> IC3C4
- DIY-305-4 pad 2: unconnected-(DIY-305-4-Row1-Pad2) -> IC3R1
- DIY-305-4 pad 3: unconnected-(DIY-305-4-Row3-Pad3) -> IC3R3
- DIY-305-4 pad 4: unconnected-(DIY-305-4-Row4-Pad4) -> IC3R4
- DIY-305-4 pad 5: unconnected-(DIY-305-4-Col1-Pad5) -> IC3C1
- DIY-305-4 pad 7: unconnected-(DIY-305-4-Dot-Pad7) -> IC3C8
- DIY-305-4 pad 8: unconnected-(DIY-305-4-Col3-Pad8) -> IC3C3
- DIY-305-4 pad 9: unconnected-(DIY-305-4-Row7-Pad9) -> IC3R7
- DIY-305-5 pad 1: unconnected-(DIY-305-5-Col2-Pad1) -> IC3R2
- DIY-305-5 pad 10: unconnected-(DIY-305-5-Row6-Pad10) -> IC3C6
- DIY-305-5 pad 11: unconnected-(DIY-305-5-Row5-Pad11) -> IC3C5
- DIY-305-5 pad 12: unconnected-(DIY-305-5-Row2-Pad12) -> IC3C2
- DIY-305-5 pad 13: unconnected-(DIY-305-5-Col5-Pad13) -> IC3R5
- DIY-305-5 pad 14: unconnected-(DIY-305-5-Col4-Pad14) -> IC3R4
- DIY-305-5 pad 2: unconnected-(DIY-305-5-Row1-Pad2) -> IC3C1
- DIY-305-5 pad 3: unconnected-(DIY-305-5-Row3-Pad3) -> IC3C3
- DIY-305-5 pad 4: unconnected-(DIY-305-5-Row4-Pad4) -> IC3C4
- DIY-305-5 pad 5: unconnected-(DIY-305-5-Col1-Pad5) -> IC3R1
- DIY-305-5 pad 7: unconnected-(DIY-305-5-Dot-Pad7) -> IC3R8
- DIY-305-5 pad 8: unconnected-(DIY-305-5-Col3-Pad8) -> IC3R3
- DIY-305-5 pad 9: unconnected-(DIY-305-5-Row7-Pad9) -> IC3C7
- DIY-305-6 pad 1: unconnected-(DIY-305-6-Col2-Pad1) -> IC4C2
- DIY-305-6 pad 10: unconnected-(DIY-305-6-Row6-Pad10) -> IC4R6
- DIY-305-6 pad 11: unconnected-(DIY-305-6-Row5-Pad11) -> IC4R5
- DIY-305-6 pad 12: unconnected-(DIY-305-6-Row2-Pad12) -> IC4R2
- DIY-305-6 pad 13: unconnected-(DIY-305-6-Col5-Pad13) -> IC4C5
- DIY-305-6 pad 14: unconnected-(DIY-305-6-Col4-Pad14) -> IC4C4
- DIY-305-6 pad 2: unconnected-(DIY-305-6-Row1-Pad2) -> IC4R1
- DIY-305-6 pad 3: unconnected-(DIY-305-6-Row3-Pad3) -> IC4R3
- DIY-305-6 pad 4: unconnected-(DIY-305-6-Row4-Pad4) -> IC4R4
- DIY-305-6 pad 5: unconnected-(DIY-305-6-Col1-Pad5) -> IC4C1
- DIY-305-6 pad 7: unconnected-(DIY-305-6-Dot-Pad7) -> IC4C8
- DIY-305-6 pad 8: unconnected-(DIY-305-6-Col3-Pad8) -> IC4C3
- DIY-305-6 pad 9: unconnected-(DIY-305-6-Row7-Pad9) -> IC4R7
- DIY-305-7 pad 1: unconnected-(DIY-305-7-Col2-Pad1) -> IC4R2
- DIY-305-7 pad 10: unconnected-(DIY-305-7-Row6-Pad10) -> IC4C6
- DIY-305-7 pad 11: unconnected-(DIY-305-7-Row5-Pad11) -> IC4C5
- DIY-305-7 pad 12: unconnected-(DIY-305-7-Row2-Pad12) -> IC4C2
- DIY-305-7 pad 13: unconnected-(DIY-305-7-Col5-Pad13) -> IC4R5
- DIY-305-7 pad 14: unconnected-(DIY-305-7-Col4-Pad14) -> IC4R4
- DIY-305-7 pad 2: unconnected-(DIY-305-7-Row1-Pad2) -> IC4C1
- DIY-305-7 pad 3: unconnected-(DIY-305-7-Row3-Pad3) -> IC4C3
- DIY-305-7 pad 4: unconnected-(DIY-305-7-Row4-Pad4) -> IC4C4
- DIY-305-7 pad 5: unconnected-(DIY-305-7-Col1-Pad5) -> IC4R1
- DIY-305-7 pad 7: unconnected-(DIY-305-7-Dot-Pad7) -> IC4R8
- DIY-305-7 pad 8: unconnected-(DIY-305-7-Col3-Pad8) -> IC4R3
- DIY-305-7 pad 9: unconnected-(DIY-305-7-Row7-Pad9) -> IC4C7
Routing:
- net PB0: track 57.1 -> 134.9 mm, vias 2 -> 7
- net PB2: track 55.9 -> 127.9 mm, vias 3 -> 8
- net VCC: track 0.00 -> 58.2 mm, vias 0 -> 4
- net +3V3: track 66.7 -> 121.4 mm, vias 2 -> 7
- net VBUS: track 18.8 -> 58.2 mm, vias 2 -> 3

Commit message: let autorouter go crazy
Parts:
- removed C12, C13, C6, C7: 0402 1uF, Capacitor_SMD:C_0402_1005Metric
- added C16: 0402 0.1uF, Capacitor_SMD:C_0402_1005Metric, F.Cu at (66.5, 47.1)
- added C17: 0402 1uF, Capacitor_SMD:C_0402_1005Metric, F.Cu at (66.5, 46.1)
- added C18: 0402 10uF, Capacitor_SMD:C_0402_1005Metric, F.Cu at (66.5, 45.1)
- added R0: 10K 0402, Resistor_SMD:R_0402_1005Metric, F.Cu at (52.0, 33.7)
- added R10: 10K 0402, Resistor_SMD:R_0402_1005Metric, F.Cu at (60.1, 33.7)
- added R11: 10K 0402, Resistor_SMD:R_0402_1005Metric, F.Cu at (70.2, 33.8)
- added R12: 10K 0402, Resistor_SMD:R_0402_1005Metric, F.Cu at (69.2, 33.8)
- added R13: 10K 0402, Resistor_SMD:R_0402_1005Metric, F.Cu at (56.2, 56.5)
- added R14: 10K 0402, Resistor_SMD:R_0402_1005Metric, F.Cu at (56.2, 55.5)
- added R15: 10K 0402, Resistor_SMD:R_0402_1005Metric, F.Cu at (30.5, 56.5)
- added R16: 10K 0402, Resistor_SMD:R_0402_1005Metric, F.Cu at (30.5, 55.5)
- added R6: 10K 0402, Resistor_SMD:R_0402_1005Metric, F.Cu at (51.0, 33.8)
- added R7: 10K 0402, Resistor_SMD:R_0402_1005Metric, F.Cu at (42.8, 33.7)
- added R8: 10K 0402, Resistor_SMD:R_0402_1005Metric, F.Cu at (41.7, 33.7)
- added R9: 10K 0402, Resistor_SMD:R_0402_1005Metric, F.Cu at (61.1, 33.7)
- added U0: TCA9548ARGER, Package_DFN_QFN:Texas_RGE0024C_EP2.1x2.1mm, F.Cu at (66.8, 50.3)
- moved C9 21.7 mm to (65.4, 38.8)
- moved C15 21.7 mm to (56.5, 38.8)
- moved C14 21.7 mm to (74.6, 38.8)
- moved C8 21.7 mm to (47.1, 38.8)
- moved C5 21.4 mm to (65.4, 37.8)
- moved IC4 21.4 mm to (73.4, 34.5)
- moved C11 21.4 mm to (56.5, 37.8)
- moved IC1 21.4 mm to (45.9, 34.5)
- moved IC2 21.4 mm to (55.3, 34.5)
- moved C0 21.4 mm to (47.1, 37.8)
- moved C10 21.4 mm to (74.6, 37.8)
- moved IC3 21.4 mm to (64.2, 34.5)
Connections:
- IC1 pad 1: PB0 -> SDA2_3V3
- IC1 pad 2: PB2 -> SCL2_3V3
- IC2 pad 1: PB0 -> SDA3_3V3
- IC2 pad 2: PB2 -> SCL3_3V3
- IC2 pad 6: PB0 -> SDA3_3V3
- IC3 pad 1: PB0 -> SDA4_3V3
- IC3 pad 2: PB2 -> SCL4_3V3
- IC3 pad 6: PB2 -> SCL4_3V3
- IC4 pad 1: PB0 -> SDA5_3V3
- IC4 pad 2: PB2 -> SCL5_3V3
- U1 pad 10: PB0 -> SDA1_3V3
- U1 pad 9: PB2 -> SCL1_3V3
- U2 pad 1: PB0 -> SDA0_3V3
- U2 pad 6: PB2 -> SCL0_3V3
Routing:
- net IC2R3: track 0.00 -> 154.5 mm, vias 0 -> 2
- net IC2C3: track 0.00 -> 146.1 mm, vias 0 -> 2
- net IC2C5: track 0.00 -> 142.1 mm, vias 0 -> 2
- net IC2R2: track 0.00 -> 140.0 mm, vias 0 -> 3
- net IC2C7: track 0.00 -> 134.4 mm, vias 0 -> 3
- net IC2R4: track 0.00 -> 130.6 mm, vias 0 -> 3
- net IC2C8: track 0.00 -> 121.3 mm, vias 0 -> 2
- net IC2R1: track 0.00 -> 121.1 mm, vias 0 -> 3
- net IC2C6: track 0.00 -> 117.2 mm, vias 0 -> 3
- net IC2R5: track 0.00 -> 113.8 mm, vias 0 -> 3
- net IC2C1: track 0.00 -> 104.6 mm, vias 0 -> 2
- net IC2C2: track 0.00 -> 97.4 mm, vias 0 -> 2
- net IC2C4: track 0.00 -> 92.8 mm, vias 0 -> 1
- net IC4R5: track 0.00 -> 78.3 mm, vias 0 -> 1
- net IC4R2: track 0.00 -> 77.0 mm, vias 0 -> 3
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
Commit message: clearanced the matrix
Routing:
- net IC4R2: track 77.0 -> 81.0 mm
- net IC1C4: track 23.5 -> 26.6 mm
- net IC4C2: track 61.5 -> 64.0 mm
- net IC2C1: track 104.6 -> 107.1 mm
- net IC4C4: track 49.0 -> 51.2 mm
- net IC2C5: track 142.1 -> 144.1 mm
- net IC2R2: track 140.0 -> 141.9 mm
- net IC3C2: track 47.4 -> 49.2 mm
- net IC4C3: track 42.6 -> 44.3 mm
- net IC3R1: track 41.8 -> 43.3 mm
- net IC2R3: track 154.5 -> 156.0 mm
- net IC2C4: track 92.8 -> 94.2 mm
- net IC3C4: track 30.4 -> 31.8 mm
- net IC3R2: track 44.8 -> 46.0 mm
- net IC2C2: track 97.4 -> 98.6 mm
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
Commit message: generated production files
Parts:
- removed C1: 10nF 0402, Capacitor_SMD:C_0402_1005Metric
- added C_BYP_1: 10nF 0402, Capacitor_SMD:C_0402_1005Metric, F.Cu at (37.6, 50.0)
- J1: value USB_C_Receptacle_USB2.0_16P -> HRO_TYPE-C-31-M-12
- U3: value SPX3819DIY-305-5-L-3-3 -> LDO SOT-23-5 3.3V
Routing:
- net IC2R4: track 131.3 -> 148.1 mm
- net IC2R2: track 141.9 -> 153.4 mm
- net IC2C3: track 147.3 -> 153.3 mm
- net IC2C7: track 135.4 -> 139.0 mm
- net IC2C8: track 121.3 -> 123.4 mm
- net IC2R3: track 156.0 -> 157.3 mm
- net IC2C6: track 118.0 -> 118.9 mm

Commit message: updated production files and silkscreen
Routing:
- net IC2C7: track 139.0 -> 149.3 mm
- net IC2C8: track 123.4 -> 130.7 mm
- net IC2R3: track 157.3 -> 163.0 mm
- net IC2R4: track 148.1 -> 149.3 mm

Commit message: began re-work on fixing colossal mistakes
Parts:
- removed C0, C10, C11, C5: 0402 0.1uF, Capacitor_SMD:C_0402_1005Metric
- removed C14, C15, C8, C9: 0402 10uF, Capacitor_SMD:C_0402_1005Metric
- removed R0, R10, R11, R12, R6, R7, R8, R9: 10K 0402, Resistor_SMD:R_0402_1005Metric
- added C101: 0402 0.1uF, Capacitor_SMD:C_0402_1005Metric, F.Cu at (28.1, 39.6)
- added C102: 0402 1uF, Capacitor_SMD:C_0402_1005Metric, F.Cu at (28.1, 40.6)
- added C103: 0402 10uF, Capacitor_SMD:C_0402_1005Metric, F.Cu at (28.1, 41.5)
- added C104: 0402 0.1uF, Capacitor_SMD:C_0402_1005Metric, F.Cu at (50.1, 39.6)
- added C105: 0402 1uF, Capacitor_SMD:C_0402_1005Metric, F.Cu at (50.1, 40.6)
- added C106: 0402 10uF, Capacitor_SMD:C_0402_1005Metric, F.Cu at (50.1, 41.6)
- added C107: 0402 0.1uF, Capacitor_SMD:C_0402_1005Metric, F.Cu at (72.1, 39.6)
- added C108: 0402 1uF, Capacitor_SMD:C_0402_1005Metric, F.Cu at (72.1, 40.6)
- added C109: 0402 10uF, Capacitor_SMD:C_0402_1005Metric, F.Cu at (72.1, 41.6)
- added C110: 0402 0.1uF, Capacitor_SMD:C_0402_1005Metric, F.Cu at (94.1, 39.6)
- added C111: 0402 1uF, Capacitor_SMD:C_0402_1005Metric, F.Cu at (94.1, 40.6)
- added C112: 0402 10uF, Capacitor_SMD:C_0402_1005Metric, F.Cu at (94.1, 41.6)
- added R101: 10K 0402, Resistor_SMD:R_0402_1005Metric, F.Cu at (22.6, 36.3)
- added R102: 10K 0402, Resistor_SMD:R_0402_1005Metric, F.Cu at (21.6, 36.3)
- added R103: 10K 0402, Resistor_SMD:R_0402_1005Metric, F.Cu at (44.6, 36.2)
- added R104: 10K 0402, Resistor_SMD:R_0402_1005Metric, F.Cu at (43.6, 36.2)
- added R105: 10K 0402, Resistor_SMD:R_0402_1005Metric, F.Cu at (66.6, 36.3)
- added R106: 10K 0402, Resistor_SMD:R_0402_1005Metric, F.Cu at (65.6, 36.3)
- added R107: 10K 0402, Resistor_SMD:R_0402_1005Metric, F.Cu at (88.6, 36.3)
- added R108: 10K 0402, Resistor_SMD:R_0402_1005Metric, F.Cu at (87.6, 36.3)
- moved IC4 19.5 mm to (92.8, 36.5)
- moved IC1 19.2 mm to (26.8, 36.5)
- moved IC3 6.82 mm to (70.8, 36.5)
- moved IC2 6.82 mm to (48.8, 36.5)
- moved NT0 3.46 mm to (56.2, 43.2)
- renumbered DIY-305-0 to DIY-305-1, DIY-305-1 to DIY-305-2, DIY-305-2 to DIY-305-3, DIY-305-3 to DIY-305-4, DIY-305-4 to DIY-305-5, DIY-305-5 to DIY-305-6, DIY-305-6 to DIY-305-7, DIY-305-7 to DIY-305-8
Connections:
- DIY-305-1 pad 1: IC2C2 -> IC1C2
- DIY-305-1 pad 10: IC2R6 -> IC1R6
- DIY-305-1 pad 11: IC2R5 -> IC1R5
- DIY-305-1 pad 12: IC2R2 -> IC1R2
- DIY-305-1 pad 13: IC2C5 -> IC1C5
- DIY-305-1 pad 14: IC2C4 -> IC1C4
- DIY-305-1 pad 2: IC2R1 -> IC1R1
- DIY-305-1 pad 3: IC2R3 -> IC1R3
- DIY-305-1 pad 4: IC2R4 -> IC1R4
- DIY-305-1 pad 5: IC2C1 -> IC1C1
- DIY-305-1 pad 7: IC2C8 -> IC1C8
- DIY-305-1 pad 8: IC2C3 -> IC1C3
- DIY-305-1 pad 9: IC2R7 -> IC1R7
- DIY-305-2 pad 1: IC2R2 -> IC1R2
- DIY-305-2 pad 10: IC2C6 -> IC1C6
- DIY-305-2 pad 11: IC2C5 -> IC1C5
- DIY-305-2 pad 12: IC2C2 -> IC1C2
- DIY-305-2 pad 13: IC2R5 -> IC1R5
- DIY-305-2 pad 14: IC2R4 -> IC1R4
- DIY-305-2 pad 2: IC2C1 -> IC1C1
- DIY-305-2 pad 3: IC2C3 -> IC1C3
- DIY-305-2 pad 4: IC2C4 -> IC1C4
- DIY-305-2 pad 5: IC2R1 -> IC1R1
- DIY-305-2 pad 7: IC2R8 -> IC1R8
- DIY-305-2 pad 8: IC2R3 -> IC1R3
- DIY-305-2 pad 9: IC2C7 -> IC1C7
- DIY-305-3 pad 1: IC1C2 -> IC2C2
- DIY-305-3 pad 10: IC1R6 -> IC2R6
- DIY-305-3 pad 11: IC1R5 -> IC2R5
- DIY-305-3 pad 12: IC1R2 -> IC2R2
- DIY-305-3 pad 13: IC1C5 -> IC2C5
- DIY-305-3 pad 14: IC1C4 -> IC2C4
- DIY-305-3 pad 2: IC1R1 -> IC2R1
- DIY-305-3 pad 3: IC1R3 -> IC2R3
- DIY-305-3 pad 4: IC1R4 -> IC2R4
- DIY-305-3 pad 5: IC1C1 -> IC2C1
- DIY-305-3 pad 7: IC1C8 -> IC2C8
- DIY-305-3 pad 8: IC1C3 -> IC2C3
- DIY-305-3 pad 9: IC1R7 -> IC2R7
- DIY-305-4 pad 1: IC1R2 -> IC2R2
- DIY-305-4 pad 10: IC1C6 -> IC2C6
- DIY-305-4 pad 11: IC1C5 -> IC2C5
- DIY-305-4 pad 12: IC1C2 -> IC2C2
- DIY-305-4 pad 13: IC1R5 -> IC2R5
- DIY-305-4 pad 14: IC1R4 -> IC2R4
- DIY-305-4 pad 2: IC1C1 -> IC2C1
- DIY-305-4 pad 3: IC1C3 -> IC2C3
- DIY-305-4 pad 4: IC1C4 -> IC2C4
- DIY-305-4 pad 5: IC1R1 -> IC2R1
- DIY-305-4 pad 7: IC1R8 -> IC2R8
- DIY-305-4 pad 8: IC1R3 -> IC2R3
- DIY-305-4 pad 9: IC1C7 -> IC2C7
- IC1 pad 1: SDA2_3V3 -> SDA7_3V3
- IC1 pad 2: SCL2_3V3 -> SCL7_3V3
- IC2 pad 1: SDA3_3V3 -> SDA6_3V3
- IC2 pad 10: IC3R4 -> IC2R4
- IC2 pad 12: IC3R5 -> IC2R5
- IC2 pad 13: IC3R6 -> IC2R6
- IC2 pad 14: IC3R7 -> IC2R7
- IC2 pad 15: IC3R8 -> IC2R8
- IC2 pad 16: IC3C8 -> IC2C8
- IC2 pad 17: IC3C7 -> IC2C7
- IC2 pad 18: IC3C6 -> IC2C6
- IC2 pad 19: IC3C5 -> IC2C5
- IC2 pad 2: SCL3_3V3 -> SCL6_3V3
- IC2 pad 21: IC3C4 -> IC2C4
- IC2 pad 22: IC3C3 -> IC2C3
- IC2 pad 23: IC3C2 -> IC2C2
- IC2 pad 24: IC3C1 -> IC2C1
- IC2 pad 6: SDA3_3V3 -> GND
- IC2 pad 7: IC3R1 -> IC2R1
- IC2 pad 8: IC3R2 -> IC2R2
- IC2 pad 9: IC3R3 -> IC2R3
- IC3 pad 1: SDA4_3V3 -> SDA5_3V3
- IC3 pad 10: IC4R4 -> IC3R4
- IC3 pad 12: IC4R5 -> IC3R5
- IC3 pad 13: IC4R6 -> IC3R6
- IC3 pad 14: IC4R7 -> IC3R7
- IC3 pad 15: IC4R8 -> IC3R8
- IC3 pad 16: IC4C8 -> IC3C8
- IC3 pad 17: IC4C7 -> IC3C7
- IC3 pad 18: IC4C6 -> IC3C6
- IC3 pad 19: IC4C5 -> IC3C5
- IC3 pad 2: SCL4_3V3 -> SCL5_3V3
- IC3 pad 21: IC4C4 -> IC3C4
- IC3 pad 22: IC4C3 -> IC3C3
- IC3 pad 23: IC4C2 -> IC3C2
- IC3 pad 24: IC4C1 -> IC3C1
- IC3 pad 6: SCL4_3V3 -> SDA5_3V3
- IC3 pad 7: IC4R1 -> IC3R1
- IC3 pad 8: IC4R2 -> IC3R2
- IC3 pad 9: IC4R3 -> IC3R3
- IC4 pad 1: SDA5_3V3 -> SDA4_3V3
- IC4 pad 10: IC2R4 -> IC4R4
- IC4 pad 12: IC2R5 -> IC4R5
- IC4 pad 13: IC2R6 -> IC4R6
- IC4 pad 14: IC2R7 -> IC4R7
- IC4 pad 15: IC2R8 -> IC4R8
- IC4 pad 16: IC2C8 -> IC4C8
- IC4 pad 17: IC2C7 -> IC4C7
- IC4 pad 18: IC2C6 -> IC4C6
- IC4 pad 19: IC2C5 -> IC4C5
- IC4 pad 2: SCL5_3V3 -> SCL4_3V3
- IC4 pad 21: IC2C4 -> IC4C4
- IC4 pad 22: IC2C3 -> IC4C3
- IC4 pad 23: IC2C2 -> IC4C2
- IC4 pad 24: IC2C1 -> IC4C1
- IC4 pad 6: GND -> SCL4_3V3
- IC4 pad 7: IC2R1 -> IC4R1
- IC4 pad 8: IC2R2 -> IC4R2
- IC4 pad 9: IC2R3 -> IC4R3
Routing:
- net IC2R3: track 163.0 -> 0.00 mm, vias 2 -> 0
- net IC2R2: track 153.8 -> 0.00 mm, vias 3 -> 0
- net IC2C3: track 153.3 -> 0.00 mm, vias 2 -> 0
- net IC2C7: track 149.3 -> 0.00 mm, vias 3 -> 0
- net IC2R4: track 149.3 -> 0.00 mm, vias 3 -> 0
- net IC2C5: track 144.6 -> 0.00 mm, vias 2 -> 0
- net IC2C8: track 130.7 -> 0.00 mm, vias 2 -> 0
- net IC2R1: track 121.8 -> 0.00 mm, vias 3 -> 0
- net IC2C6: track 118.9 -> 0.00 mm, vias 3 -> 0
- net IC2R5: track 114.6 -> 0.00 mm, vias 3 -> 0
- net IC2C1: track 107.1 -> 0.00 mm, vias 2 -> 0
- net IC2C2: track 98.6 -> 0.00 mm, vias 2 -> 0
- net IC2C4: track 94.2 -> 0.00 mm, vias 1 -> 0
- net IC4R2: track 81.0 -> 0.00 mm, vias 3 -> 0
- net IC4R5: track 79.2 -> 0.00 mm, vias 1 -> 0
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
Commit message: re-did the PCB
Routing:
- net SCL7_3V3: track 0.00 -> 92.8 mm, vias 0 -> 2
- net VCC: track 12.7 -> 85.6 mm
- net +3V3: track 84.8 -> 157.2 mm, vias 3 -> 8
- net SDA7_3V3: track 0.00 -> 64.0 mm, vias 0 -> 2
- net IC1R2: track 0.00 -> 56.9 mm, vias 0 -> 1
- net IC4R4: track 0.00 -> 56.5 mm, vias 0 -> 1
- net IC4R2: track 0.00 -> 50.6 mm, vias 0 -> 1
- net IC3C2: track 0.00 -> 50.5 mm
- net IC1R3: track 0.00 -> 50.1 mm, vias 0 -> 3
- net IC2R4: track 0.00 -> 50.1 mm, vias 0 -> 1
- net IC3R4: track 0.00 -> 49.9 mm
- net IC1R4: track 0.00 -> 48.4 mm, vias 0 -> 2
- net IC1C2: track 0.00 -> 45.5 mm
- net IC2R3: track 0.00 -> 44.6 mm, vias 0 -> 3
- net IC4R5: track 0.00 -> 44.0 mm
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
Commit message: generated production files
Routing:
- net IC1R7: track 12.9 -> 13.5 mm
- net GND: vias 65 -> 68
Changed lines of the file:
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@@
   (via (at 21.825 20.2) (size 0.4) (drill 0.2) (layers "F.Cu" "B.Cu") (free) (net 2))
   (via (at 43.75 26.325) (size 0.8) (drill 0.4) (layers "F.Cu" "B.Cu") (free) (net 2))
+  (via (at 33.525 33.8) (size 0.8) (drill 0.4) (layers "F.Cu" "B.Cu") (free) (net 2))
   (via (at 60.55 40.55) (size 0.8) (drill 0.4) (layers "F.Cu" "B.Cu") (free) (net 2))
+  (via (at 31.175 28.25) (size 0.8) (drill 0.4) (layers "F.Cu" "B.Cu") (free) (net 2))
   (via (at 24.5 34.125) (size 0.8) (drill 0.4) (layers "F.Cu" "B.Cu") (free) (net 2))
   (via (at 64.2 26.125) (size 0.8) (drill 0.4) (layers "F.Cu" "B.Cu") (free) (net 2))
@@
   (via (at 21.325 26.8) (size 0.4) (drill 0.2) (layers "F.Cu" "B.Cu") (free) (net 2))
   (via (at 55.025 32.15) (size 0.8) (drill 0.4) (layers "F.Cu" "B.Cu") (free) (net 2))
+  (via (at 33.85 38.825) (size 0.8) (drill 0.4) (layers "F.Cu" "B.Cu") (free) (net 2))
   (via (at 85.8 39.125) (size 0.4) (drill 0.2) (layers "F.Cu" "B.Cu") (free) (net 2))
   (via (at 99.85 37.3) (size 0.8) (drill 0.4) (layers "F.Cu" "B.Cu") (free) (net 2))
@@
   (segment (start 29.6996 37.2873) (end 28.7248 37.2873) (width 0.15) (layer "F.Cu") (net 28))
   (segment (start 28.7248 37.2873) (end 28.6875 37.25) (width 0.15) (layer "F.Cu") (net 28))
-  (segment (start 26.4 28.655) (end 26.4 31.2961) (width 0.15) (layer "F.Cu") (net 28))
-  (segment (start 25.07 27.325) (end 26.4 28.655) (width 0.15) (layer "F.Cu") (net 28))
-  (via (at 26.4 31.2961) (size 0.4) (drill 0.2) (layers "F.Cu" "B.Cu") (net 28))
+  (segment (start 26.575 32.475) (end 26.575 28.83) (width 0.15) (layer "F.Cu") (net 28))
+  (segment (start 26.575 28.83) (end 25.07 27.325) (width 0.15) (layer "F.Cu") (net 28))
+  (via (at 26.575 32.475) (size 0.4) (drill 0.2) (layers "F.Cu" "B.Cu") (net 28))
   (via (at 29.6996 37.2873) (size 0.4) (drill 0.2) (layers "F.Cu" "B.Cu") (net 28))
-  (segment (start 26.4 31.2961) (end 29.6996 34.5957) (width 0.15) (layer "B.Cu") (net 28))
+  (segment (start 26.575 32.475) (end 27.5789 32.475) (width 0.15) (layer "B.Cu") (net 28))
+  (segment (start 27.5789 32.475) (end 29.6996 34.5957) (width 0.15) (layer "B.Cu") (net 28))
   (segment (start 29.6996 34.5957) (end 29.6996 37.2873) (width 0.15) (layer "B.Cu") (net 28))
   (segment (start 28.7923 37.8548) (end 30.4316 37.8548) (width 0.15) (layer "F.Cu") (net 29))
   (segment (start 28.6875 37.75) (end 28.7923 37.8548) (width 0.15) (layer "F.Cu") (net 29))
   (via (at 30.4316 37.8548) (size 0.4) (drill 0.2) (layers "F.Cu" "B.Cu") (net 29))
-  (segment (start 24.05375 25.80125) (end 24.05375 26.70375) (width 0.15) (layer "B.Cu") (net 29))
-  (segment (start 25.07 24.785) (end 24.05375 25.80125) (width 0.15) (layer "B.Cu") (net 29))
+  (segment (start 24.2743 37.0305) (end 23.1725 35.9287) (width 0.15) (layer "B.Cu") (net 29))
+  (segment (start 23.1725 35.9287) (end 23.1725 27.585) (width 0.15) (layer "B.Cu") (net 29))
+  (segment (start 29.3029 37.8548) (end 28.9081 38.2496) (width 0.15) (layer "B.Cu") (net 29))
   (segment (start 23.1725 27.585) (end 24.05375 26.70375) (width 0.15) (layer "B.Cu") (net 29))
-  (segment (start 24.2743 37.0305) (end 23.1725 35.9287) (width 0.15) (layer "B.Cu") (net 29))
+  (segment (start 24.05375 26.70375) (end 24.05375 25.80125) (width 0.15) (layer "B.Cu") (net 29))
+  (segment (start 24.05375 25.80125) (end 25.07 24.785) (width 0.15) (layer "B.Cu") (net 29))
+  (segment (start 28.9081 38.2496) (end 25.036864 38.2496) (width 0.15) (layer "B.Cu") (net 29))
+  (segment (start 25.036864 38.2496) (end 24.2743 37.487036) (width 0.15) (layer "B.Cu") (net 29))
+  (segment (start 24.2743 37.487036) (end 24.2743 37.0305) (width 0.15) (layer "B.Cu") (net 29))
   (segment (start 30.4316 37.8548) (end 29.3029 37.8548) (width 0.15) (layer "B.Cu") (net 29))
-  (segment (start 23.1725 35.9287) (end 23.1725 27.585) (width 0.15) (layer "B.Cu") (net 29))
-  (segment (start 29.3029 37.8548) (end 29.031 38.1267) (width 0.15) (layer "B.Cu") (net 29))
-  (segment (start 25.2341 38.1267) (end 24.2743 37.1669) (width 0.15) (layer "B.Cu") (net 29))
-  (segment (start 24.2743 37.1669) (end 24.2743 37.0305) (width 0.15) (layer "B.Cu") (net 29))
-  (segment (start 29.031 38.1267) (end 25.2341 38.1267) (width 0.15) (layer "B.Cu") (net 29))
   (segment (start 30.3747 39.5257) (end 37.45 32.4504) (width 0.15) (layer "F.Cu") (net 30))
   (segment (start 28 38.4375) (end 28.5241 38.4375) (width 0.15) (layer "F.Cu") (net 30))
