File: EnvOpenSensor-ATTINY/MCU.kicad_sch (KiCad schematic)
At the start: 5 parts, among them J3 AVR-ISP-6, U5 ATtiny1634-M

Commit message: added pullup to reset (schematic only)
Parts:
- added R6: 10K 0402, Resistor_SMD:R_0402_1005Metric, symbol Device:R_Small
Connections:
- net +3V3: now also R6.2
- net PC3: now also R6.1
Changed lines of the file:
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@@
 	(wire
 		(pts
-			(xy 73.025 109.22) (xy 68.58 109.22)
+			(xy 77.47 109.22) (xy 68.58 109.22)
 		)
 		(stroke
@@
 		(pts
 			(xy 69.85 152.4) (xy 66.04 152.4)
+		)
+		(stroke
+			(width 0)
+			(type default)
+		)
+	)
+	(wire
+		(pts
+			(xy 90.424 109.22) (xy 82.55 109.22)
 		)
 		(stroke
@@
 	(symbol
 		(lib_id "power:+3V3")
+		(at 90.424 109.22 0)
+		(unit 1)
+		(exclude_from_sim no)
+		(in_bom yes)
+		(on_board yes)
+		(dnp no)
+		(fields_autoplaced yes)
+		(property "Reference" "#PWR049"
+			(at 90.424 113.03 0)
+			(effects
+				(font
+					(size 1.27 1.27)
+				)
+				(hide yes)
+			)
+		)
+		(property "Value" "+3V3"
+			(at 90.424 104.14 0)
+			(effects
+				(font
+					(size 1.27 1.27)
+				)
+			)
+		)
+		(property "Footprint" ""
+			(at 90.424 109.22 0)
+			(effects
+				(font
+					(size 1.27 1.27)
+				)
+				(hide yes)
+			)
+		)
+		(property "Datasheet" ""
+			(at 90.424 109.22 0)
+			(effects
+				(font
+					(size 1.27 1.27)
+				)
+				(hide yes)
+			)
+		)
+		(property "Description" "Power symbol creates a global label with name \"+3V3\""
+			(at 90.424 109.22 0)
+			(effects
+				(font
+					(size 1.27 1.27)
+				)
+				(hide yes)
+			)
+		)
+		(pin "1"
+		)
+		(instances
+			(project "EnvOpenSensor"
+				(path "/2bbc1dac-4f9d-46a0-a466-6585abe7fd58/ed2ce937-d069-4d0b-9c23-efb500873d25"
+					(reference "#PWR049")
+					(unit 1)
+				)
+			)
+		)
+	)
+	(symbol
+		(lib_id "power:+3V3")
 		(at 53.34 142.24 0)
 		(unit 1)
@@
 					(unit 1)
 				)
+			)
+		)
+	)
+	(symbol
+		(lib_id "Device:R_Small")
+		(at 80.01 109.22 90)
+		(unit 1)
+		(exclude_from_sim no)
+		(in_bom yes)
+		(on_board yes)
+		(dnp no)
+		(property "Reference" "R6"
+			(at 80.01 110.998 90)
+			(effects
+				(font
+					(size 0.635 0.635)
+				)
+				(justify top)
+			)
+		)
+		(property "Value" "10K 0402"
+			(at 80.01 108.204 90)
+			(effects
+				(font
+					(size 0.635 0.635)
+				)
+				(justify top)
+			)
+		)
+		(property "Footprint" "Resistor_SMD:R_0402_1005Metric"
+			(at 80.01 109.22 0)
+			(effects
+				(font
+					(size 1.27 1.27)
+				)
+				(hide yes)
+			)
+		)
+		(property "Datasheet" "~"
+			(at 80.01 109.22 0)
+			(effects
+				(font
+					(size 1.27 1.27)
+				)
+				(hide yes)
+			)
+		)
+		(property "Description" "Resistor, small symbol"
+			(at 80.01 109.22 0)
+			(effects
+				(font
+					(size 1.27 1.27)
+				)
+				(hide yes)
+			)
+		)
+		(pin "2"
+		)
+		(pin "1"
+		)
+		(instances
+			(project ""
+				(path "/2bbc1dac-4f9d-46a0-a466-6585abe7fd58/ed2ce937-d069-4d0b-9c23-efb500873d25"
+					(reference "R6")
+					(unit 1)
+				)
